File: v2/schematic_smd.sch (EAGLE design)
At the start: 16 parts, among them J2 DCJ0202, U1 328P

Commit message: Added v2 smd board
Parts:
- removed C2: 22pF, SparkFun-Capacitors:22PF-PTH-2.54MM-200V-5%
- removed R1: 10k, SparkFun-Resistors:10KOHM-HORIZ-1/4W-1%
- removed R2, R3: 220, SparkFun-Resistors:10KOHM-HORIZ-1/4W-1%
- removed R4: 470ohm, SparkFun-Resistors:10KOHM-HORIZ-1/4W-1%
- added C3, C5: 22pF, SparkFun-Capacitors:1.0UF-1206-50V-10%
- added R5: 10k, SparkFun-Resistors:0.22OHM-0805-1/4W-1%
- added R6: 1k, SparkFun-Resistors:10OHM-1206-1/4W-1%
- added R7, R8: 470, SparkFun-Resistors:10OHM-1206-1/4W-1%
- C1: value 22pF -> 1uF; device SparkFun-Capacitors:22PF-PTH-2.54MM-200V-5% -> SparkFun-Capacitors:1.0UF-1206-50V-10%
- LEDS: value (none) -> Leds; device SparkFun-Connectors:CONN_02 -> SparkFun-Connectors:CONN_02JST-PTH-2-KIT
- USB: device SparkFun-Connectors:CONN_02 -> SparkFun-Connectors:CONN_02JST-PTH-2-KIT
Connections:
- net 12VO: now also C1.1
- net GND: now also C1.2, C3.1, C4.+, C5.1, R7.1, USB.1; no longer C1.1, C2.1, C4.-, R3.1, USB.2
- net N$1: now also C5.2; no longer C1.2
- net N$2: now also C3.2; no longer C2.2
- net N$3: now also R6.2; no longer R2.2
- net N$4: now also R8.2; no longer R4.2
- net PIN12: now also R8.1; no longer R4.1
- net PIN2: now also R7.2; no longer R3.2
- net PIN8: now also R6.1; no longer R2.1
- net RESET: now also R5.2; no longer R1.2
- net VCC: now also C4.-, R5.1, USB.2; no longer C4.+, R1.1, USB.1
Other:
- moved on the sheet: C1
